File: 6s_750mA/6s_750mA.kicad_sch (KiCad schematic)
At the start: 2 parts, among them J1 Barrel_Jack_MountingPin, J2 S6B-XH-A

Commit message: fix supplier part numbers for power connector and battery connector
Parts:
- J1: Manufacturer Part Number PJ-002A -> PJ-102AH; Supplier Part Number CP-002A-ND -> CP-102AH-ND
- J2: Manufacturer Part Number S6B-XH-A -> S7B-XH-A; Supplier Part Number 455-S6B-XH-A-ND -> 455-S7B-XH-A-ND
Changed lines of the file:
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@@
       (effects (font (size 1.27 1.27)) hide)
     )
-    (property "Datasheet" "https://www.cuidevices.com/product/resource/pj-002a.pdf" (at 53.34 91.186 0)
+    (property "Datasheet" "https://www.cuidevices.com/product/resource/pj-102ah.pdf" (at 53.34 91.186 0)
       (effects (font (size 1.27 1.27)) hide)
     )
@@
       (effects (font (size 1.27 1.27)) hide)
     )
-    (property "Supplier Part Number" "CP-002A-ND" (at 52.07 90.17 0)
+    (property "Supplier Part Number" "CP-102AH-ND" (at 52.07 90.17 0)
       (effects (font (size 1.27 1.27)) hide)
     )
-    (property "Manufacturer Part Number" "PJ-002A" (at 52.07 90.17 0)
+    (property "Manufacturer Part Number" "PJ-102AH" (at 52.07 90.17 0)
       (effects (font (size 1.27 1.27)) hide)
     )
@@
       (effects (font (size 1.27 1.27)) hide)
     )
-    (property "Supplier Part Number" "455-S6B-XH-A-ND" (at 132.08 92.71 0)
+    (property "Supplier Part Number" "455-S7B-XH-A-ND" (at 132.08 92.71 0)
       (effects (font (size 1.27 1.27)) hide)
     )
-    (property "Manufacturer Part Number" "S6B-XH-A" (at 132.08 92.71 0)
+    (property "Manufacturer Part Number" "S7B-XH-A" (at 132.08 92.71 0)
       (effects (font (size 1.27 1.27)) hide)
     )
